File: Backplane/Backplane.sch (EAGLE design)
At the start: 14 parts, among them X1 FAC64S, X2 FAC64S, X3 FAC64S, X4 FAC64S, X5 FAC64S, X6 FAC64S, X7 FAC64S, X9 5566-20

Commit message: Fixed fit between backplane & enclosure
Parts:
- R1: value 220 -> (none)
Changed lines of the file:
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@@
 <part name="S1" library="SparkFun-Electromechanical" deviceset="SWITCH-SPDT" device="PTH"/>
 <part name="LED1" library="SparkFun-LED" deviceset="LED" device="3MM"/>
-<part name="R1" library="SparkFun-Passives" deviceset="RESISTOR" device="KIT" value="220"/>
+<part name="R1" library="SparkFun-Passives" deviceset="RESISTOR" device="KIT"/>
 <part name="JP3" library="SparkFun-Connectors" deviceset="M03" device="LONGPADS"/>
 <part name="X9" library="con-molex" deviceset="5566-20" device=""/>
