File: RAM Board/RAM Board Deux.sch (EAGLE design)
At the start: 24 parts, among them IC1 74LS32N, IC2 74LS04N, IC3 74LS138N, IC6 74LS32N, U1 AS6C4008, U2 AS6C4008, U3 AS6C4008, U4 AS6C4008, U5 AS6C4008, U6 AS6C4008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

Commit message: Built breakout board and RAM card
Parts:
- removed C11, C4, C5: 100nF, SparkFun-Capacitors:CAPPTH
- removed IC1, IC6: 74LS32N, 74xx-us:74LS32N
- removed IC2: 74LS04N, 74xx-eu:74LS04N
- removed IC3: 74LS138N, 74xx-eu:74LS138N
- added JP36, JP37, JP38, JP39: M01PTH, SparkFun-Connectors:M01PTH
- added U$2: M191X19_NO_SILK, SparkFun-Connectors:M191X19_NO_SILK
Connections:
- removed net /BOOT: IC6A.I0, IC6B.I0, IC6C.I0, IC6D.I0
- removed net N$18: IC3A.Y6, IC6A.I1
- removed net N$20: IC3A.Y4, IC6C.I1
- removed net N$22: IC3A.Y2, IC6D.I1
- removed net N$24: IC3A.Y0, IC6B.I1
- removed net N$3: IC1A.I1, IC1B.I1, IC2A.O
- net /AS: no longer IC3A.A
- net /LDS: no longer IC1B.I0, IC1D.I0
- net /UDS: no longer IC1A.I0, IC1C.I0
- net ADDRESS0: now also U$2.1
- net ADDRESS1: now also U$2.2
- net ADDRESS10: now also U$2.11
- net ADDRESS11: now also U$2.12
- net ADDRESS12: now also U$2.13
- net ADDRESS13: now also U$2.14
- net ADDRESS14: now also U$2.15
- net ADDRESS15: now also U$2.16
- net ADDRESS16: now also U$2.17
- net ADDRESS17: now also U$2.18
- net ADDRESS18: now also U$2.19
- net ADDRESS2: now also U$2.3
- net ADDRESS20: no longer IC3A.B
- net ADDRESS21: no longer IC3A.C
- net ADDRESS3: now also U$2.4
- net ADDRESS4: now also U$2.5
- net ADDRESS5: now also U$2.6
- net ADDRESS6: now also U$2.7
- net ADDRESS7: now also U$2.8
- net ADDRESS8: now also U$2.9
- net ADDRESS9: now also U$2.10
- net BANKACS: now also JP39.1; no longer IC6B.O
- net BANKBCS: now also JP38.1; no longer IC6D.O
- net BANKCCS: now also JP37.1; no longer IC6C.O
- net BANKDCS: now also JP36.1; no longer IC6A.O
- net GND: no longer C11.2, C4.2, C5.2, IC3A.G2A, IC3A.G2B
- net R/W: no longer IC1C.I1, IC1D.I1, IC2A.I
- net READHI: no longer IC1A.O
- net READLO: no longer IC1B.O
- net VCC: no longer C11.1, C4.1, C5.1, IC3A.G1
- net WRITEHI: no longer IC1C.O
- net WRITELO: no longer IC1D.O
